File: docs/track-a/eda/GridUp-Modul.kicad_sch (KiCad schematic)
At the start: 54 parts, among them J1 İç ihtiyaç L / N / PE, J2 CT L1, J3 CT L2, J4 CT L3, J5 CT nötr, J6 Genişleme 2×5, J7 RS-485 klemens B / GND / A, J8 SMA panel, J9 Servis USB/UART0, SW1 Reset, U1 ESP32-S3-WROOM-1U-N8, U2 MLX90640ESF-BAA, U3 SHT31-DIS-B, U4 MAX3485, U5 RAC05-05SK/277, U6 AP7361C-33E 3,3 V / 1 A, U7 TPS61099 4,6 V

Commit message: İZ A: 03 — V_bias notu '3V3/2 = 1,65 V (CT DC ofseti)'
Other:
- note added: "V_bias = 3V3/2 = 1,65 V (CT DC ofseti)"
- note removed: "V_bias = 3V3/2 (CT ön yargı)"
Changed lines of the file:
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@@
 		)
 	)
-	(text "V_bias = 3V3/2 (CT ön yargı)"
+	(text "V_bias = 3V3/2 = 1,65 V (CT DC ofseti)"
 		(exclude_from_sim no)
 		(at 66.04 121.92 0)

Commit message: İZ A: 03 — V_bias notu '3,3 V / 2 = 1,65 V'
Other:
- note added: "V_bias = 3,3 V / 2 = 1,65 V (CT DC ofseti)"
- note removed: "V_bias = 3V3/2 = 1,65 V (CT DC ofseti)"
Changed lines of the file:
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@@
 		)
 	)
-	(text "V_bias = 3V3/2 = 1,65 V (CT DC ofseti)"
+	(text "V_bias = 3,3 V / 2 = 1,65 V (CT DC ofseti)"
 		(exclude_from_sim no)
 		(at 66.04 121.92 0)

Commit message: İZ A: 03 — V_bias notu '3V3 / 2 = 1,65 V'
Other:
- note added: "V_bias = 3V3 / 2 = 1,65 V (CT DC ofseti)"
- note removed: "V_bias = 3,3 V / 2 = 1,65 V (CT DC ofseti)"
Changed lines of the file:
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@@
 		)
 	)
-	(text "V_bias = 3,3 V / 2 = 1,65 V (CT DC ofseti)"
+	(text "V_bias = 3V3 / 2 = 1,65 V (CT DC ofseti)"
 		(exclude_from_sim no)
 		(at 66.04 121.92 0)
